File: AirBoxnano.kicad_pcb (KiCad board)
At the start: 2 copper layers, 44 x 21 mm, 37 parts, among them P1 CONN_01X14, P2 CONN_01X08, P3 CONN_01X15, P4 CONN_01X15, P5 CONN_01X02, U1 ATmega32U4-AU, U2 NCP1117ST33T3G, U3 SHT20, Y1 16MHz

Commit message: update readme
Parts:
- removed P5: CONN_01X02, Connectors:CONN_2.54mm_1x2
- added D1: GREEN, LEDs:LED_0603, F.Cu at (56.4, 51.9)
- added D2: MBR120, AirBox:SOD-323, F.Cu at (86.7, 69.7)
- added R7: 10K, Resistors_SMD:R_0603, F.Cu at (67.7, 51.3)
- added R8: 10K, Resistors_SMD:R_0603, F.Cu at (52.0, 66.1)
- added SW1: SW, AirBoxnano:SW_SPDT, B.Cu at (90.0, 67.1)
- added U4: AP2112-3.3, TO_SOT_Packages_SMD:SOT-23-5, F.Cu at (55.2, 66.2)
- C3: value 22uF -> 10uF; footprint Capacitors_Tantalum_SMD:TantalC_SizeA_EIA-3216_Wave -> Capacitors_SMD:C_0603
- C5: value 100nF -> 10uF
- C7: value 10uF/25V -> 10uF; footprint Capacitors_Tantalum_SMD:TantalC_SizeA_EIA-3216_Wave -> Capacitors_SMD:C_0603
- C8: value 10uF -> 1uF
- P3: value CONN_01X15 -> BATT; footprint AirBoxnano:CONN_2.54mm_1x15 -> AirBoxnano:BATconn
- P4: value CONN_01X15 -> CONN_01X06; footprint AirBoxnano:CONN_2.54mm_1x15 -> Connectors:CONN_2.54mm_1x6
- R4: value 10K -> 1K
- U2: value NCP1117ST33T3G -> MCP73831; footprint TO_SOT_Packages_SMD:SOT-223 -> TO_SOT_Packages_SMD:SOT-23-5
- U3: footprint Housings_DFN_QFN:DFN-6-1EP_3x3mm_Pitch0.95mm -> AirBoxnano:DFN-6-1EP_3x3mm_Pitch0.95mm
- moved C3 28.7 mm to (83.3, 69.7), turned to 180 degrees
- moved D3 26.4 mm to (73.6, 51.4), turned to 0 degrees
- moved P3 23.6 mm to (91.9, 69.2), turned to 90 degrees
- moved R9 22.7 mm to (76.6, 51.4), turned to 0 degrees
- moved C8 16.7 mm to (58.9, 65.2)
- moved U2 15.7 mm to (63.9, 52.3), turned to 0 degrees
- moved R4 15.5 mm to (60.1, 51.3)
- moved C5 12.0 mm to (67.9, 53.1), turned to 0 degrees
- moved C12 9.67 mm to (55.0, 63.1)
- moved C10 6.76 mm to (60.8, 56.0), turned to 180 degrees
- moved C13 6.37 mm to (58.5, 63.1), turned to 0 degrees
- moved C7 5.46 mm to (59.0, 67.2), turned to 0 degrees
- moved P4 3.41 mm to (58.0, 69.5), turned to 0 degrees
- moved R12 3.31 mm to (63.6, 64.5), turned to 0 degrees
- moved C11 3.24 mm to (63.8, 66.3), turned to 0 degrees
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Connections:
- C3 pad 1: +5C -> Net-(C3-Pad1)
- C5 pad 1: GND -> +5C
- C5 pad 2: +5C -> GND
- C6 pad 2: +5C -> +3V3
- C7 pad 1: +5C -> +3V3
- LED1 pad 1: +5C -> /A0
- P2 pad 8: +5C -> /A0
- P3 pad 1: /A0 -> +5C
- P3 pad 2: /A1 -> GND
- P4 pad 1: GND -> /MISO
- P4 pad 3: +3V3 -> /SCK
- P4 pad 4: +5C -> /MOSI
- P4 pad 5: GND -> /RESET
- P4 pad 6: /D0 -> GND
- R1 pad 2: +5C -> +3V3
- R4 pad 1: GND -> Net-(R4-Pad1)
- R4 pad 2: +5C -> Net-(D1-Pad1)
- U1 pad 14: +5C -> +3V3
- U1 pad 2: +5C -> +3V3
- U1 pad 24: +5C -> +3V3
- U1 pad 34: +5C -> +3V3
- U1 pad 44: +5C -> +3V3
- U1 pad 6: +5C -> +3V3
- U2 pad 1: GND -> Net-(R4-Pad1)
- U2 pad 2: +3V3 -> GND
- U2 pad 4: (no net) -> +5C
Routing:
- net +5C: track 123.3 -> 55.0 mm, vias 3 -> 2
- net /A0: track 8.96 -> 63.2 mm, vias 0 -> 3
- net +3V3: track 98.1 -> 137.4 mm, vias 3 -> 4
- net /D7: track 24.0 -> 0.00 mm, vias 1 -> 0
- net /AREF: track 28.2 -> 4.29 mm, vias 1 -> 0
- net /IO8: track 14.8 -> 0.00 mm, vias 1 -> 0
- net /D0: track 14.8 -> 0.00 mm, vias 1 -> 0
- net /IO11: track 14.4 -> 0.00 mm
- net /IO9: track 14.1 -> 0.00 mm, vias 1 -> 0
- net /MOSI: track 10.3 -> 23.3 mm
- net /IO10: track 12.8 -> 0.00 mm, vias 1 -> 0
- net /D1: track 12.6 -> 0.00 mm, vias 1 -> 0
- net /A5: track 10.7 -> 0.00 mm, vias 1 -> 0
- net /A4: track 10.5 -> 0.00 mm, vias 1 -> 0
- net /A3: track 8.68 -> 0.00 mm, vias 1 -> 0
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Other:
- board text added: "AirBoxnano"
- board text added: "G"
- board text added: "R"
- board text added: "S"
- board text added: "V"
- board text added: "v0.2"
- board text removed: "-"
- board text removed: "3V3"
- board text removed: "5V"
- board text removed: "A0"
- board text removed: "A1"
- board text removed: "A2"
- board text removed: "A3"
- board text removed: "A4"
- board text removed: "A5"
- board text removed: "AREF"
- board text removed: "D0"
- board text removed: "D1"
- board text removed: "D10"
- board text removed: "D11"
- board text removed: "D12"
- board text removed: "D13"
- board text removed: "D7"
- board text removed: "D8"
- board text removed: "D9"
- board text removed: "GND"
- board text removed: "RES"
- board text removed: "SCK"
- board text removed: "SCL"
- board text removed: "SDA"

Commit message: del temp/hum
Parts:
- removed C15: 0.1uF, Capacitors_SMD:C_0603
- removed D2: MBR120, AirBox:SOD-323
- removed D3: L, LEDs:LED_0603
- removed P4: CONN_01X06, Connectors:CONN_2.54mm_1x6
- removed R11, R9: 1K, Resistors_SMD:R_0603
- removed R12: 820K, Resistors_SMD:R_0603
- removed R13: 10K, Resistors_SMD:R_0603
- removed SW1: SW, AirBoxnano:SW_SPDT
- removed U3: SHT20, AirBoxnano:DFN-6-1EP_3x3mm_Pitch0.95mm
- removed U4: AP2112-3.3, TO_SOT_Packages_SMD:SOT-23-5
- added REF***: OSHW-Logo2_7.3x6mm_SilkScreen, Symbols:OSHW-Logo2_7.3x6mm_SilkScreen, B.Cu at (89.9, 54.3)
- C3: value 10uF -> 22uF; footprint Capacitors_SMD:C_0603 -> Capacitors_Tantalum_SMD:Tantalum_Case-A_EIA-3216-18_Reflow
- C5: value 10uF -> 100nF
- C7: value 10uF -> 10uF/25V; footprint Capacitors_SMD:C_0603 -> Capacitors_Tantalum_SMD:Tantalum_Case-A_EIA-3216-18_Reflow
- C8: value 1uF -> 10uF
- D1: value GREEN -> L
- P3: value BATT -> CONN_01X06; footprint AirBoxnano:BATconn -> Connectors:CONN_2.54mm_1x6
- R4: value 1K -> 10K
- R5, R6: value 10K -> 1K
- R7: value 10K -> 820K
- U2: value MCP73831 -> NCP1117ST33T3G; footprint TO_SOT_Packages_SMD:SOT-23-5 -> TO_SOT_Packages_SMD:SOT-223
- moved D1 40.0 mm to (92.1, 70.0), turned to 180 degrees
- moved P3 34.3 mm to (57.6, 69.8), turned to 0 degrees
- moved C3 29.4 mm to (58.7, 53.6), turned to 0 degrees
- moved R8 20.4 mm to (67.0, 52.3)
- moved C11 16.3 mm to (72.3, 52.4), turned to 90 degrees
- moved U2 15.7 mm to (54.6, 65.0), turned to 90 degrees
- moved R5 14.6 mm to (89.1, 70.0), turned to 180 degrees
- moved C6 12.8 mm to (74.1, 52.4)
- moved R6 11.5 mm to (86.1, 67.1)
- moved C9 10.9 mm to (64.1, 65.5)
- moved C10 10.4 mm to (70.6, 52.4), turned to 90 degrees
- moved C12 9.34 mm to (61.9, 56.8), turned to 270 degrees
- moved C13 8.11 mm to (63.6, 56.8), turned to 270 degrees
- moved C5 7.71 mm to (60.4, 51.3), turned to 180 degrees
- moved C8 5.54 mm to (64.1, 67.1)
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Connections:
- C3 pad 1: Net-(C3-Pad1) -> +5C
- C5 pad 1: +5C -> GND
- C5 pad 2: GND -> +5C
- C7 pad 1: +3V3 -> +5C
- D1 pad 1: Net-(D1-Pad1) -> GND
- D1 pad 2: +5C -> Net-(D1-Pad2)
- LED1 pad 1: /A0 -> +5C
- P2 pad 4: /D4 -> /IO8
- P2 pad 5: /D5 -> Net-(P2-Pad5)
- P2 pad 8: /A0 -> +5C
- P3 pad 1: +5C -> /MISO
- P3 pad 2: GND -> +3V3
- R1 pad 2: +3V3 -> +5C
- R4 pad 1: Net-(R4-Pad1) -> GND
- R4 pad 2: Net-(D1-Pad1) -> +5C
- R5 pad 1: +3V3 -> Net-(D1-Pad2)
- R5 pad 2: /D2 -> /IO13
- R6 pad 1: +3V3 -> GND
- R6 pad 2: /D3 -> /HWB
- R7 pad 1: GND -> Net-(P1-Pad12)
- R7 pad 2: Net-(R7-Pad2) -> GND
- R8 pad 1: Net-(R8-Pad1) -> /RES
- R8 pad 2: /A0 -> +3V3
- U2 pad 1: Net-(R4-Pad1) -> GND
- U2 pad 2: GND -> +3V3
- U2 pad 4: +5C -> (no net)
Routing:
- net /A0: track 63.2 -> 0.00 mm, vias 3 -> 0
- net +3V3: track 137.4 -> 80.5 mm, vias 4 -> 3
- net /D2: track 52.5 -> 22.8 mm
- net /D3: track 47.4 -> 24.5 mm
- net /D4: track 16.6 -> 0.00 mm, vias 2 -> 0
- net /IO8: track 0.00 -> 12.6 mm
- net GND: track 214.5 -> 202.1 mm, vias 9 -> 11
- net /D5: track 11.1 -> 0.00 mm, vias 2 -> 0
- net +5C: track 55.0 -> 64.4 mm
- net Net-(C11-Pad1): track 6.15 -> 13.0 mm
- net Net-(P1-Pad12): track 4.15 -> 10.8 mm
- net Net-(C10-Pad1): track 5.16 -> 11.6 mm
- net Net-(C13-Pad1): track 4.71 -> 9.82 mm
- net /D6: track 16.6 -> 21.6 mm, vias 0 -> 2
- net Net-(C12-Pad1): track 4.19 -> 9.14 mm
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Other:
- board text added: "-"
- board text added: "3V3"
- board text added: "Airboxnano v0.3"
- board text added: "GND"
- board text added: "RESET"
- board text added: "SCK"
- board text added: "https://github.com/danfei/AirBoxnano"
- board text removed: "AirBoxnano"
- board text removed: "G"
- board text removed: "R"
- board text removed: "S"
- board text removed: "V"
- board text removed: "v0.2"
