File: AirBoxnano.sch (KiCad schematic (older format))
At the start: 37 parts, among them P1 CONN_01X14, P2 CONN_01X08, P3 CONN_01X15, P4 CONN_01X15, P5 CONN_01X02, U1 ATmega32U4-AU, U2 NCP1117ST33T3G, U3 SHT20, Y1 16MHz

Commit message: update sch
Parts:
- removed C3: 22uF, Capacitors_Tantalum_SMD:TantalC_SizeA_EIA-3216_Wave, symbol CP_Small
- removed C5: 100nF, Capacitors_SMD:C_0603, symbol C_Small
- removed C7: 10uF/25V, Capacitors_Tantalum_SMD:TantalC_SizeA_EIA-3216_Wave, symbol CP1_Small
- removed C8: 10uF, Capacitors_SMD:C_0603, symbol C_Small
- removed P3, P4: CONN_01X15, AirBoxnano:CONN_2.54mm_1x15, symbol CONN_01X15
- removed P5: CONN_01X02, Connectors:CONN_2.54mm_1x2, symbol CONN_01X02
- removed R4: 10K, Resistors_SMD:R_0603, symbol R_Small
- removed U2: NCP1117ST33T3G, TO_SOT_Packages_SMD:SOT-223, symbol NCP1117ST33T3G
- added C? (x3): 10uF, Capacitors_SMD:C_0603, symbol C_Small
- added C?: 1uF, Capacitors_SMD:C_0603, symbol C_Small
- added D?: MBR120, symbol D_Small
- added D?: GREEN, symbol LED_Small
- added P?: BATT, symbol CONN_01X02
- added R? (x2): 10K, Resistors_SMD:R_0603, symbol R_Small
- added R?: 1K, Resistors_SMD:R_0603, symbol R_Small
- added SW?: SW, symbol SW
- added U?: AP2112-3.3, symbol AP2112-3.3
- added U?: MCP73831, symbol MCP73831
Connections:
- net labels added: +BATT, VOL
- wire segments 178 -> 162
- no-connect marks 8 -> 9

Commit message: update footprint
Parts:
- D1: renamed from D?; footprint (none) -> LEDs:LED_0603
- D2: renamed from D?; footprint (none) -> AirBox:SOD-323
- P3: renamed from P?; footprint (none) -> AirBoxnano:BATconn
- SW1: renamed from SW?; footprint (none) -> AirBoxnano:SW_SPDT
- U2, U4: renamed from U?; footprint (none) -> TO_SOT_Packages_SMD:SOT-23-5
- gave numbers to parts that had none: 7

Commit message: update readme
Parts:
- added P4: CONN_01X06, Connectors:CONN_2.54mm_1x6, symbol CONN_01X06
- U3: footprint Housings_DFN_QFN:DFN-6-1EP_3x3mm_Pitch0.95mm -> AirBoxnano:DFN-6-1EP_3x3mm_Pitch0.95mm
Connections:
- net labels removed: +5V
- wire segments 162 -> 170
Changed lines of the file:
@@
 $EndComp
 $Comp
-L GND #PWR01
+L GND #PWR2
 U 1 1 57202D44
 P 1250 1475
-F 0 "#PWR01" H 1250 1225 50  0001 C CNN
+F 0 "#PWR2" H 1250 1225 50  0001 C CNN
 F 1 "GND" H 1250 1325 50  0000 C CNN
 F 2 "" H 1250 1475 50  0000 C CNN
@@
 $EndComp
 $Comp
-L GND #PWR02
+L GND #PWR9
 U 1 1 572031EC
 P 2200 4125
-F 0 "#PWR02" H 2200 3875 50  0001 C CNN
+F 0 "#PWR9" H 2200 3875 50  0001 C CNN
 F 1 "GND" H 2200 3975 50  0000 C CNN
 F 2 "" H 2200 4125 50  0000 C CNN
@@
 D-
 $Comp
-L VBUS #PWR03
+L VBUS #PWR6
 U 1 1 57203841
 P 1750 1725
-F 0 "#PWR03" H 1750 1575 50  0001 C CNN
+F 0 "#PWR6" H 1750 1575 50  0001 C CNN
 F 1 "VBUS" H 1750 1865 50  0000 C CNN
 F 2 "" H 1750 1725 50  0000 C CNN
@@
 $EndComp
 $Comp
-L GND #PWR04
+L GND #PWR1
 U 1 1 572040D7
 P 950 3325
-F 0 "#PWR04" H 950 3075 50  0001 C CNN
+F 0 "#PWR1" H 950 3075 50  0001 C CNN
 F 1 "GND" H 950 3175 50  0000 C CNN
 F 2 "" H 950 3325 50  0000 C CNN
@@
 $EndComp
 $Comp
-L GND #PWR05
+L GND #PWR28
 U 1 1 57206BC1
 P 7075 5300
-F 0 "#PWR05" H 7075 5050 50  0001 C CNN
+F 0 "#PWR28" H 7075 5050 50  0001 C CNN
 F 1 "GND" H 7075 5150 50  0000 C CNN
 F 2 "" H 7075 5300 50  0000 C CNN
@@
 $EndComp
 $Comp
-L GND #PWR06
+L GND #PWR4
 U 1 1 57207539
 P 1500 4725
-F 0 "#PWR06" H 1500 4475 50  0001 C CNN
+F 0 "#PWR4" H 1500 4475 50  0001 C CNN
 F 1 "GND" H 1500 4575 50  0000 C CNN
 F 2 "" H 1500 4725 50  0000 C CNN
@@
 D-
 $Comp
-L VBUS #PWR07
+L VBUS #PWR7
 U 1 1 57207BAB
 P 1850 5425
-F 0 "#PWR07" H 1850 5275 50  0001 C CNN
+F 0 "#PWR7" H 1850 5275 50  0001 C CNN
 F 1 "VBUS" H 1850 5565 50  0000 C CNN
 F 2 "" H 1850 5425 50  0000 C CNN
@@
 $EndComp
 $Comp
-L GND #PWR08
+L GND #PWR24
 U 1 1 5880A0B2
 P 6275 2625
-F 0 "#PWR08" H 6275 2375 50  0001 C CNN
+F 0 "#PWR24" H 6275 2375 50  0001 C CNN
 F 1 "GND" H 6275 2475 50  0000 C CNN
 F 2 "" H 6275 2625 50  0000 C CNN
@@
 $EndComp
 $Comp
-L GND #PWR09
+L GND #PWR23
 U 1 1 5880A0B3
 P 6100 1825
-F 0 "#PWR09" H 6100 1575 50  0001 C CNN
+F 0 "#PWR23" H 6100 1575 50  0001 C CNN
 F 1 "GND" H 6100 1675 50  0000 C CNN
 F 2 "" H 6100 1825 50  0000 C CNN
@@
 SDA
 $Comp
-L +3V3 #PWR010
+L +3V3 #PWR26
 U 1 1 5880A0B4
 P 7050 2900
-F 0 "#PWR010" H 7050 2750 50  0001 C CNN
+F 0 "#PWR26" H 7050 2750 50  0001 C CNN
 F 1 "+3V3" H 7050 3040 50  0000 C CNN
 F 2 "" H 7050 2900 50  0000 C CNN
@@
 $EndComp
 $Comp
-L GND #PWR011
+L GND #PWR27
 U 1 1 5880A0B7
 P 7050 3500
-F 0 "#PWR011" H 7050 3250 50  0001 C CNN
+F 0 "#PWR27" H 7050 3250 50  0001 C CNN
 F 1 "GND" H 7050 3350 50  0000 C CNN
 F 2 "" H 7050 3500 50  0000 C CNN
@@
 RES
 $Comp
-L +3V3 #PWR012
+L +3V3 #PWR25
 U 1 1 5880A0BB
 P 6500 3225
-F 0 "#PWR012" H 6500 3075 50  0001 C CNN
+F 0 "#PWR25" H 6500 3075 50  0001 C CNN
 F 1 "+3V3" H 6500 3365 50  0000 C CNN
 F 2 "" H 6500 3225 50  0000 C CNN
@@
 SCL
 $Comp
-L +3V3 #PWR013
+L +3V3 #PWR22
 U 1 1 5880A0BE
 P 6050 1625
-F 0 "#PWR013" H 6050 1475 50  0001 C CNN
+F 0 "#PWR22" H 6050 1475 50  0001 C CNN
 F 1 "+3V3" H 6050 1765 50  0000 C CNN
 F 2 "" H 6050 1625 50  0000 C CNN
@@
 F 0 "U3" H 8800 3250 60  0000 C CNN
 F 1 "SHT20" H 8550 3250 60  0000 C CNN
-F 2 "Housings_DFN_QFN:DFN-6-1EP_3x3mm_Pitch0.95mm" H 8675 3250 60  0001 C CNN
+F 2 "AirBoxnano:DFN-6-1EP_3x3mm_Pitch0.95mm" H 8675 3250 60  0001 C CNN
 F 3 "" H 8675 3250 60  0001 C CNN
 	1    8675 3400
@@
 $EndComp
 $Comp
-L GND #PWR014
+L GND #PWR29
 U 1 1 5880B460
 P 8125 3600
-F 0 "#PWR014" H 8125 3350 50  0001 C CNN
+F 0 "#PWR29" H 8125 3350 50  0001 C CNN
 F 1 "GND" H 8125 3450 50  0000 C CNN
 F 2 "" H 8125 3600 50  0000 C CNN
@@
 $EndComp
 $Comp
-L +3V3 #PWR015
+L +3V3 #PWR33
 U 1 1 5880C3FE
 P 9150 3000
-F 0 "#PWR015" H 9150 2850 50  0001 C CNN
+F 0 "#PWR33" H 9150 2850 50  0001 C CNN
 F 1 "+3V3" H 9150 3140 50  0000 C CNN
 F 2 "" H 9150 3000 50  0000 C CNN
@@
 $EndComp
 $Comp
-L +5V #PWR016
-U 1 1 5880E0E8
-P 8925 4500
-F 0 "#PWR016" H 8925 4350 50  0001 C CNN
-F 1 "+5V" H 8925 4640 50  0000 C CNN
-F 2 "" H 8925 4500 50  0000 C CNN
-F 3 "" H 8925 4500 50  0000 C CNN
-	1    8925 4500
-	1    0    0    -1
-$EndComp
-$Comp
-L GND #PWR017
+L GND #PWR30
 U 1 1 5880E315
 P 8475 4775
-F 0 "#PWR017" H 8475 4525 50  0001 C CNN
+F 0 "#PWR30" H 8475 4525 50  0001 C CNN
 F 1 "GND" H 8475 4625 50  0000 C CNN
 F 2 "" H 8475 4775 50  0000 C CNN
@@
 $EndComp
 $Comp
-L +5V #PWR018
-U 1 1 5880FB0A
-P 9475 3625
-F 0 "#PWR018" H 9475 3475 50  0001 C CNN
-F 1 "+5V" H 9475 3765 50  0000 C CNN
-F 2 "" H 9475 3625 50  0000 C CNN
-F 3 "" H 9475 3625 50  0000 C CNN
-	1    9475 3625
-	1    0    0    -1
-$EndComp
-$Comp
-L GND #PWR019
+L GND #PWR34
 U 1 1 5880FF57
 P 10500 4100
-F 0 "#PWR019" H 10500 3850 50  0001 C CNN
+F 0 "#PWR34" H 10500 3850 50  0001 C CNN
 F 1 "GND" H 10500 3950 50  0000 C CNN
 F 2 "" H 10500 4100 50  0000 C CNN
@@
 	9625 3800 9250 3800
 Wire Wire Line
-	9625 3700 9475 3700
-Wire Wire Line
-	8925 4700 8925 4500
+	9475 3700 9625 3700
 Wire Wire Line
 	8475 4775 8475 4600
@@
 	2200 975  2200 2075
 Wire Wire Line
-	9475 3700 9475 3625
+	9475 3575 9475 3700
 Wire Wire Line
 	8475 4600 8350 4600
@@
 NoConn ~ 8350 4000
 $Comp
-L +3V3 #PWR020
+L +3V3 #PWR8
 U 1 1 58B2843E
 P 2200 975
-F 0 "#PWR020" H 2200 825 50  0001 C CNN
+F 0 "#PWR8" H 2200 825 50  0001 C CNN
 F 1 "+3V3" H 2200 1115 50  0000 C CNN
 F 2 "" H 2200 975 50  0000 C CNN
@@
 $EndComp
 $Comp
-L +3V3 #PWR021
+L +3V3 #PWR5
 U 1 1 58B288C5
 P 1600 2125
-F 0 "#PWR021" H 1600 1975 50  0001 C CNN
+F 0 "#PWR5" H 1600 1975 50  0001 C CNN
 F 1 "+3V3" H 1600 2265 50  0000 C CNN
 F 2 "" H 1600 2125 50  0000 C CNN
@@
 	1250 5525 1250 5225
 $Comp
-L VBUS #PWR022
+L VBUS #PWR10
 U 1 1 58B298C5
 P 2450 4750
-F 0 "#PWR022" H 2450 4600 50  0001 C CNN
+F 0 "#PWR10" H 2450 4600 50  0001 C CNN
 F 1 "VBUS" H 2450 4890 50  0000 C CNN
 F 2 "" H 2450 4750 50  0000 C CNN
@@
 $EndComp
 $Comp
-L +BATT #PWR023
+L +BATT #PWR11
 U 1 1 58B29910
 P 2700 4750
-F 0 "#PWR023" H 2700 4600 50  0001 C CNN
+F 0 "#PWR11" H 2700 4600 50  0001 C CNN
 F 1 "+BATT" H 2700 4890 50  0000 C CNN
 F 2 "" H 2700 4750 50  0000 C CNN
@@
 $EndComp
 $Comp
-L +3V3 #PWR024
+L +3V3 #PWR18
 U 1 1 58B2A3FD
 P 4600 4750
-F 0 "#PWR024" H 4600 4600 50  0001 C CNN
+F 0 "#PWR18" H 4600 4600 50  0001 C CNN
 F 1 "+3V3" H 4600 4890 50  0000 C CNN
 F 2 "" H 4600 4750 50  0000 C CNN
@@
 $EndComp
 $Comp
-L GND #PWR025
+L GND #PWR12
 U 1 1 58B2A5F6
 P 2700 5400
-F 0 "#PWR025" H 2700 5150 50  0001 C CNN
+F 0 "#PWR12" H 2700 5150 50  0001 C CNN
 F 1 "GND" H 2700 5250 50  0000 C CNN
 F 2 "" H 2700 5400 50  0000 C CNN
@@
 $EndComp
 $Comp
-L GND #PWR026
+L GND #PWR16
 U 1 1 58B2A673
 P 3400 5150
-F 0 "#PWR026" H 3400 4900 50  0001 C CNN
+F 0 "#PWR16" H 3400 4900 50  0001 C CNN
 F 1 "GND" H 3400 5000 50  0000 C CNN
 F 2 "" H 3400 5150 50  0000 C CNN
@@
 $EndComp
 $Comp
-L GND #PWR027
+L GND #PWR17
 U 1 1 58B2A6F0
 P 4400 5200
-F 0 "#PWR027" H 4400 4950 50  0001 C CNN
+F 0 "#PWR17" H 4400 4950 50  0001 C CNN
 F 1 "GND" H 4400 5050 50  0000 C CNN
 F 2 "" H 4400 5200 50  0000 C CNN
@@
 $EndComp
 $Comp
-L GND #PWR028
+L GND #PWR19
 U 1 1 58B2A76D
 P 4600 5200
-F 0 "#PWR028" H 4600 4950 50  0001 C CNN
+F 0 "#PWR19" H 4600 4950 50  0001 C CNN
 F 1 "GND" H 4600 5050 50  0000 C CNN
 F 2 "" H 4600 5200 50  0000 C CNN
@@
 $EndComp
 $Comp
-L +BATT #PWR029
+L +BATT #PWR20
 U 1 1 58B2BE3E
 P 5300 4750
-F 0 "#PWR029" H 5300 4600 50  0001 C CNN
+F 0 "#PWR20" H 5300 4600 50  0001 C CNN
 F 1 "+BATT" H 5300 4890 50  0000 C CNN
 F 2 "" H 5300 4750 50  0000 C CNN
@@
 $EndComp
 $Comp
-L GND #PWR030
+L GND #PWR21
 U 1 1 58B2BF81
 P 5300 5100
-F 0 "#PWR030" H 5300 4850 50  0001 C CNN
+F 0 "#PWR21" H 5300 4850 50  0001 C CNN
 F 1 "GND" H 5300 4950 50  0000 C CNN
 F 2 "" H 5300 5100 50  0000 C CNN
@@
 $EndComp
 $Comp
-L VBUS #PWR031
+L VBUS #PWR3
 U 1 1 58B2C9AE
 P 1400 6200
-F 0 "#PWR031" H 1400 6050 50  0001 C CNN
+F 0 "#PWR3" H 1400 6050 50  0001 C CNN
 F 1 "VBUS" H 1400 6340 50  0000 C CNN
 F 2 "" H 1400 6200 50  0000 C CNN
@@
 $EndComp
 $Comp
-L GND #PWR032
+L GND #PWR13
 U 1 1 58B2D720
 P 2950 6600
-F 0 "#PWR032" H 2950 6350 50  0001 C CNN
+F 0 "#PWR13" H 2950 6350 50  0001 C CNN
 F 1 "GND" H 2950 6450 50  0000 C CNN
 F 2 "" H 2950 6600 50  0000 C CNN
@@
 $EndComp
 $Comp
-L GND #PWR033
+L GND #PWR15
 U 1 1 58B2DA00
 P 3100 6600
-F 0 "#PWR033" H 3100 6350 50  0001 C CNN
+F 0 "#PWR15" H 3100 6350 50  0001 C CNN
 F 1 "GND" H 3100 6450 50  0000 C CNN
 F 2 "" H 3100 6600 50  0000 C CNN
@@
 $EndComp
 $Comp
-L +BATT #PWR034
+L +BATT #PWR14
 U 1 1 58B2DB97
 P 3100 6200
-F 0 "#PWR034" H 3100 6050 50  0001 C CNN
+F 0 "#PWR14" H 3100 6050 50  0001 C CNN
 F 1 "+BATT" H 3100 6340 50  0000 C CNN
 F 2 "" H 3100 6200 50  0000 C CNN
@@
 Text Label 5000 3975 0    60   ~ 0
 VOL
+Text Label 9500 3575 0    60   ~ 0
+VOL
+Wire Wire Line
+	9475 3575 9700 3575
+Text Label 8650 4700 0    60   ~ 0
+VOL
+$Comp
+L CONN_01X06 P4
+U 1 1 58B365BE
+P 8100 2050
+F 0 "P4" H 8100 2400 50  0000 C CNN
+F 1 "CONN_01X06" V 8200 2050 50  0000 C CNN
+F 2 "Connectors:CONN_2.54mm_1x6" H 8100 2050 50  0000 C CNN
+F 3 "" H 8100 2050 50  0000 C CNN
+	1    8100 2050
+	-1   0    0    -1
+$EndComp
+Wire Wire Line
+	8300 1800 8800 1800
+Wire Wire Line
+	8300 1900 8900 1900
+Wire Wire Line
+	8300 2000 8800 2000
+Wire Wire Line
+	8300 2100 8800 2100
+Wire Wire Line
+	8300 2200 8800 2200
+Wire Wire Line
+	8300 2300 8900 2300
+Text Label 8350 1800 0    60   ~ 0
+MISO
+Text Label 8350 2000 0    60   ~ 0
+SCK
+Text Label 8350 2100 0    60   ~ 0
+MOSI
+Text Label 8350 2200 0    60   ~ 0
+RESET
+$Comp
+L +3V3 #PWR31
+U 1 1 58B36E45
+P 8900 1750
+F 0 "#PWR31" H 8900 1600 50  0001 C CNN
+F 1 "+3V3" H 8900 1890 50  0000 C CNN
+F 2 "" H 8900 1750 50  0000 C CNN
+F 3 "" H 8900 1750 50  0000 C CNN
+	1    8900 1750
+	1    0    0    -1
+$EndComp
+$Comp
+L GND #PWR32
+U 1 1 58B36FA0
+P 8900 2350
+F 0 "#PWR32" H 8900 2100 50  0001 C CNN
+F 1 "GND" H 8900 2200 50  0000 C CNN
+F 2 "" H 8900 2350 50  0000 C CNN
+F 3 "" H 8900 2350 50  0000 C CNN
+	1    8900 2350
+	1    0    0    -1
+$EndComp
+Wire Wire Line
+	8900 1900 8900 1750
+Wire Wire Line
+	8900 2300 8900 2350
 $EndSCHEMATC

Commit message: del temp/hum
Parts:
- removed C15: 0.1uF, Capacitors_SMD:C_0603, symbol C_Small
- removed C3, C7: 10uF, Capacitors_SMD:C_0603, symbol C_Small
- removed D1: GREEN, LEDs:LED_0603, symbol LED_Small
- removed D2: MBR120, AirBox:SOD-323, symbol D_Small
- removed P3: BATT, AirBoxnano:BATconn, symbol CONN_01X02
- removed P4: CONN_01X06, Connectors:CONN_2.54mm_1x6, symbol CONN_01X06
- removed R5, R6, R7, R8: 10K, Resistors_SMD:R_0603, symbol R_Small
- removed SW1: SW, AirBoxnano:SW_SPDT, symbol SW
- removed U2: MCP73831, TO_SOT_Packages_SMD:SOT-23-5, symbol MCP73831
- removed U3: SHT20, AirBoxnano:DFN-6-1EP_3x3mm_Pitch0.95mm, symbol SHT20
- removed U4: AP2112-3.3, TO_SOT_Packages_SMD:SOT-23-5, symbol AP2112-3.3
- added C3: 22uF, Capacitors_Tantalum_SMD:Tantalum_Case-A_EIA-3216-18_Reflow, symbol CP_Small
- added C7: 10uF/25V, Capacitors_Tantalum_SMD:Tantalum_Case-A_EIA-3216-18_Reflow, symbol CP1_Small
- added P3: CONN_01X06, Connectors:CONN_2.54mm_1x6, symbol CONN_01X06
- added U2: NCP1117ST33T3G, TO_SOT_Packages_SMD:SOT-223, symbol NCP1117ST33T3G
- C5: value 10uF -> 100nF
- C8: value 1uF -> 10uF
- R4: value 1K -> 10K
- renumbered D3 to D1, R9 to R5, R11 to R6, R12 to R7, R13 to R8
Connections:
- net labels added: +5V
- net labels removed: +BATT, VOL
- wire segments 170 -> 135
- no-connect marks 9 -> 7
