File: hardware/AirBoxnano.sch (KiCad schematic (older format))
At the start: 31 parts, among them P1 CONN_01X14, P2 CONN_01X08, P3 CONN_01X06, U1 ATmega32U4-AU, U2 NCP1117ST33T3G, Y1 16MHz

Commit message: Version 0.5
Parts:
- removed D1: L, LEDs:LED_0603, symbol Led_Small
- removed P3: CONN_01X06, Connectors:CONN_2.54mm_1x6, symbol CONN_01X06
- removed R5: 1K, Resistors_SMD:R_0603, symbol R_Small
- added P3, P4: CONN_01X14, Pin_Headers:Pin_Header_Straight_1x14_Pitch2.54mm, symbol CONN_01X14
Connections:
- net labels removed: D8
- wire segments 135 -> 154
